File: kicad/CocktailMachine/power.sch (KiCad schematic (older format))
At the start: 23 parts

Commit message: - Add decoupling for all ICs - Separate power planes from buck for noise reduction - Miscellaneous fixes
Parts:
- added C?: 1uF, symbol Device:C
- added C?: 10uF, symbol Device:C
- added L? (x2): INDUCTOR, symbol pspice:INDUCTOR
Connections:
- net +5V: now also C?.1, C?.1, L?.2; no longer C?.1, C?.1, D?.2 (A), L?.2, R?.1
- net GND: now also C?.2, C?.2, L?.2; no longer C?.2, C?.2, C?.2, C?.2, D?.2 (A), D?.2 (A), J?.1, J?.2, R?.1, U?.4 (GND), U?.8 (SYNC)
- new net +5VD: C?.1, C?.1, D?.2 (A), L?.1, L?.2, R?.1
- new net GND1: C?.2, C?.2, C?.2, C?.2, D?.2 (A), D?.2 (A), J?.1, J?.2, L?.1, R?.1, U?.4 (GND), U?.8 (SYNC)
Other:
- moved on the sheet: C?, D?, F?, J?, L?, R?, U?

Commit message: Generate footprints and netlist. Begin Layout.
Parts:
- removed J?: Barrel_Jack, symbol Connector:Barrel_Jack
- added J4: Barrel_Jack_Switch, barrel_jack:MJ-180PH, symbol Connector:Barrel_Jack_Switch
- C13, C14, C15, C16, C17, C18, C19, C20, C21: renamed from C?; footprint (none) -> Capacitor_SMD:C_0603_1608Metric
- D3: renamed from D?; footprint (none) -> Diode_SMD:D_0603_1608Metric
- D5, D6: renamed from D?; footprint (none) -> LED_THT:LED_D3.0mm
- F1: renamed from F?; footprint (none) -> Fuse:Fuse_0603_1608Metric
- L1, L2, L3: renamed from L?; footprint (none) -> Inductor_SMD:L_0603_1608Metric
- R13, R14, R15, R16: renamed from R?; footprint (none) -> Resistor_SMD:R_0603_1608Metric
- U5: renamed from U?; footprint (none) -> MCP1826S-3302E_AB:TO254P482X1024X3124-3P
- U6: renamed from U?; footprint SO-8_S_LIT -> buck_lt:LT1578CS8-PBF
- gave numbers to parts that had none: 4
Connections:
- net +12V: now also J4.1
- net GND1: now also J4.2, J4.3
